Commit message: Added vacuum gripper, effort_controller, move_group sequence, pick and drop

File: urdf/box/box.xacro (robot description, xacro)
@@ -1,36 +1,37 @@
 <?xml version="1.0"?>
  <robot xmlns:xacro="http://www.ros.org/wiki/xacro" name="simple_box">
-    <link name="object_base_link">
-    </link>
-    <joint name="object_base_joint" type="fixed">
-        <parent link="object_base_link"/>
-        <child link="object_link"/>
-        <axis xyz="0 0 1" />
-        <origin xyz="0 0 0" rpy="0 0 0"/>
-    </joint>
+	 <xacro:macro name="box_inertia" params="m x y z">
+    <inertia  ixx="${m*(y*y+z*z)/12}" ixy = "0" ixz = "0"
+      iyy="${m*(x*x+z*z)/12}" iyz = "0"
+      izz="${m*(x*x+z*z)/12}"
+    />
+   </xacro:macro>
    <link name="object_link">
      <inertial>
-       <origin xyz="0 0 0" />
-       <mass value="0.1" />
-       <inertia  ixx="0.0001" ixy="0.0"  ixz="0.0"  iyy="0.0001"  iyz="0.0"  izz="0.0001" />
+    	 <origin xyz="0 0 0" rpy="0 0 0" />
+       <mass value="0.05" />
+       <xacro:box_inertia m="0.05" x="0.1" y="0.1" z="0.05" />
      </inertial>
      <visual>
-       <origin xyz="0 0 0"/>
-       <geometry>
-         <box size="0.1 0.1 0.1" />
-        </geometry>
+   	 	 <origin xyz="0 0 0" rpy="0 0 0"/>
+    	 <geometry>
+      	 <box size="0.1 0.1 0.05" />
+    	 </geometry>
      </visual>
      <collision>
-       <origin xyz="0 0 0"/>
-       <geometry>
-         <box size="0.1 0.1 0.1" />
-       </geometry>
-     </collision>
+   	 	 <origin xyz="0 0 0" rpy="0 0 0"/>
+    	 <geometry>
+      	 <box size="0.1 0.1 0.05" />
+    	 </geometry>
+	 	 </collision>
    </link>
-   <!--gazebo reference="object_base_link">
-    <gravity>0</gravity>
-   </gazebo -->
    <gazebo reference="object_link">
      <material>Gazebo/Blue</material>
+		 <mu1>10</mu1>
+     <mu2>10</mu2>
+		 <minDepth>0.003</minDepth>
+		 <maxVel>0</maxVel>
+		 <kp>1000000.0</kp>
+  	 <kd>1.0</kd>
    </gazebo>
  </robot>

File: urdf/robot/lrmate200ic_macro.xacro (robot description, xacro)
@@ -20,6 +20,6 @@
       </collision>
 			<inertial>
-        <mass value="1"/>
-        <inertia ixx="0.001" ixy="0.0" ixz="0.0" iyy="0.001" iyz="0.0" izz="0.001"/>
+        <mass value="4.85331"/>
+        <inertia ixx ="0.000533781" iyy=".055445798" izz=".02302818052" ixy="0.00012915752" ixz ="-0.002807595" iyz = "-0.000094967"/>
       </inertial>
     </link>
@@ -39,6 +39,6 @@
       </collision>
 			<inertial>
-        <mass value="1"/>
-        <inertia ixx="0.001" ixy="0.0" ixz="0.0" iyy="0.001" iyz="0.0" izz="0.001"/>
+        <mass value = "4.85331"/>
+				<inertia ixx ="0.000533781" iyy=".055445798" izz=".02302818052" ixy="0.00012915752" ixz ="-0.002807595" iyz = "-0.000094967"/>
       </inertial>
     </link>
@@ -58,6 +58,6 @@
       </collision>
 			<inertial>
-        <mass value="1"/>
-        <inertia ixx="0.001" ixy="0.0" ixz="0.0" iyy="0.001" iyz="0.0" izz="0.001"/>
+        <mass value = "7.96646"/>
+				<inertia ixx ="0.44125720672" iyy=".42103008445" izz=".03658588308" ixy="0.000023323" ixz ="-0.01624821395" iyz = "-0.00127983617"/>
       </inertial>
     </link>
@@ -77,6 +77,6 @@
       </collision>
 			<inertial>
-        <mass value="1"/>
-        <inertia ixx="0.001" ixy="0.0" ixz="0.0" iyy="0.001" iyz="0.0" izz="0.001"/>
+        <mass value = "2.401"/>
+				<inertia ixx ="0.00709493364" iyy=".08303386" izz=".007482747" ixy="0.000062924" ixz ="0.000131383" iyz = "0.000095227"/>
       </inertial>
     </link>
@@ -96,6 +96,6 @@
       </collision>
 			<inertial>
-        <mass value="1"/>
-        <inertia ixx="0.001" ixy="0.0" ixz="0.0" iyy="0.001" iyz="0.0" izz="0.001"/>
+        <mass value = "2.89084"/>
+				<inertia ixx ="0.004863267" iyy=".19336297539" izz=".19385148073" ixy="0.00303203667" ixz ="0.000018846079" iyz = "-0.00000096841"/>
       </inertial>
     </link>
@@ -115,6 +115,6 @@
       </collision>
 			<inertial>
-        <mass value="10"/>
-        <inertia ixx="0.001" ixy="0.0" ixz="0.0" iyy="0.001" iyz="0.0" izz="0.001"/>
+        <mass value = "0.043284"/>
+				<inertia ixx ="0.00029985018" iyy=".000661879" izz=".00064231094" ixy="-0.00000439197" ixz ="-0.000000345" iyz = "-0.00000008651"/>
       </inertial>
     </link>
@@ -134,8 +134,49 @@
       </collision>
 			<inertial>
-        <mass value="1"/>
-        <inertia ixx="0.001" ixy="0.0" ixz="0.0" iyy="0.001" iyz="0.0" izz="0.001"/>
-      </inertial>
-    </link>
+        <mass value="0.1"/>
+        <inertia ixx="0.0001" ixy="0.0" ixz="0.0" iyy="0.0001" iyz="0.0" izz="0.0001"/>
+      </inertial>
+    </link>
+		<link name="${prefix}friction_plate">
+			<visual>
+				<geometry>
+					<box size="0.01 0.05 0.05"/>
+        </geometry>
+			</visual>
+      <collision>
+        <geometry>
+          <box size="0.01 0.05 0.05"/>
+        </geometry>
+        <surface>
+          <friction>
+            <ode>
+              <mu>10</mu>
+              <mu2>10</mu2>
+            </ode>
+          </friction>
+        </surface>
+        <origin rpy="0 0 0" xyz="0 0 0"/>
+      </collision>
+			<inertial>
+        <origin rpy="0 0 0" xyz="0.000000 0.000000 0.000000"/>
+      	<mass value="0.0001"/>
+      	<inertia ixx="1e-08" ixy="0" ixz="0" iyy="1e-08" iyz="0" izz="1e-08"/>
+      </inertial>
+    </link>
+	  <link name="${prefix}end_effector">
+      <visual>
+        <origin rpy="0 0 0" xyz="0 0 0"/>
+        <geometry>
+          <cylinder radius="0.005" length="0.01"/>
+        </geometry>
+        <xacro:material_fanuc_gray24 />
+      </visual>
+      <inertial>
+        <origin rpy="0 0 0" xyz="0.000000 0.000000 0.000000"/>
+      	<mass value="0.0001"/>
+      	<inertia ixx="1e-08" ixy="0" ixz="0" iyy="1e-08" iyz="0" izz="1e-08"/>
+      </inertial>
+    </link>
+		<link name="world"/>
     <!-- joints: main serial chain -->
     <joint name="${prefix}joint_1" type="revolute">
@@ -144,5 +185,6 @@
       <child link="${prefix}link_1" />
       <axis xyz="0 0 1" />
-      <limit effort="0" lower="-2.9671" upper="2.9671" velocity="6.1087" />
+      <limit effort="100" lower="-2.9671" upper="2.9671" velocity="6.1087" />
+			<dynamics damping="0.0" friction="1"/>
     </joint>
     <joint name="${prefix}joint_2" type="revolute">
@@ -151,5 +193,6 @@
       <child link="${prefix}link_2" />
       <axis xyz="0 1 0" />
-      <limit effort="0" lower="-1.0472" upper="2.4435" velocity="6.1087" />
+      <limit effort="100" lower="-1.0472" upper="2.4435" velocity="6.1087" />
+			<dynamics damping="0.0" friction="1"/>
     </joint>
     <joint name="${prefix}joint_3" type="revolute">
@@ -158,5 +201,6 @@
       <child link="${prefix}link_3" />
       <axis xyz="0 -1 0" />
-      <limit effort="0" lower="-2.4784" upper="4.0143" velocity="6.9813" />
+      <limit effort="100" lower="-2.4784" upper="4.0143" velocity="6.9813" />
+			<dynamics damping="0.0" friction="1"/>
     </joint>
     <joint name="${prefix}joint_4" type="revolute">
@@ -165,5 +209,6 @@
       <child link="${prefix}link_4"/>
       <axis xyz="-1 0 0"/>
-      <limit effort="0" lower="-3.3161" upper="3.3161" velocity="7.8540" />
+      <limit effort="100" lower="-3.3161" upper="3.3161" velocity="7.8540" />
+			<dynamics damping="0.0" friction="1"/>
     </joint>
     <joint name="${prefix}joint_5" type="revolute">
@@ -172,5 +217,6 @@
       <child link="${prefix}link_5"/>
       <axis xyz="0 -1 0"/>
-      <limit effort="0" lower="-2.0944" upper="2.0944" velocity="7.8540" />
+      <limit effort="100" lower="-2.0944" upper="2.0944" velocity="7.8540" />
+			<dynamics damping="0.0" friction="1"/>
     </joint>
     <joint name="${prefix}joint_6" type="revolute">
@@ -179,7 +225,20 @@
       <child link="${prefix}link_6"/>
       <axis xyz="-1 0 0"/>
-      <limit effort="0" lower="-6.2832" upper="6.2832" velocity="12.5664" />
-    </joint>
-		<link name="world"/>
+      <limit effort="100" lower="-6.2832" upper="6.2832" velocity="12.5664" />
+			<dynamics damping="0.0" friction="1"/>
+    </joint>
+		<joint name="${prefix}end_joint" type="revolute">
+			<origin xyz="0.021 0 0.0" rpy="0 1.5708 0"/>
+      <parent link="${prefix}link_6"/>
+      <child link="${prefix}end_effector"/>
+			<axis xyz="1 0 0" />
+      <limit effort="50" velocity="50" lower="0" upper="0" />
+			<dynamics damping="0.0" friction="1"/>
+    </joint>
+		<joint name="${prefix}friction_plate_joint" type="fixed">
+      <origin xyz="0.01 0 0" rpy="0 0 0" />
+      <parent link="${prefix}link_6" />
+      <child link="${prefix}friction_plate" />
+    </joint>
   	<joint name="fixed" type="fixed">
     	<parent link="world"/>
@@ -189,5 +248,5 @@
       <type>transmission_interface/SimpleTransmission</type>
       <joint name="${prefix}joint_1">
-        <hardwareInterface>hardware_interface/PositionJointInterface</hardwareInterface>
+        <hardwareInterface>hardware_interface/EffortJointInterface</hardwareInterface>
       </joint>
       <actuator name="${prefix}joint_1">
@@ -198,5 +257,5 @@
       <type>transmission_interface/SimpleTransmission</type>
       <joint name="${prefix}joint_2">
-        <hardwareInterface>hardware_interface/PositionJointInterface</hardwareInterface>
+        <hardwareInterface>hardware_interface/EffortJointInterface</hardwareInterface>
       </joint>
       <actuator name="${prefix}joint_2">
@@ -207,5 +266,5 @@
       <type>transmission_interface/SimpleTransmission</type>
       <joint name="${prefix}joint_3">
-        <hardwareInterface>hardware_interface/PositionJointInterface</hardwareInterface>
+        <hardwareInterface>hardware_interface/EffortJointInterface</hardwareInterface>
       </joint>
       <actuator name="${prefix}joint_3">
@@ -216,5 +275,5 @@
       <type>transmission_interface/SimpleTransmission</type>
       <joint name="${prefix}joint_4">
-        <hardwareInterface>hardware_interface/PositionJointInterface</hardwareInterface>
+        <hardwareInterface>hardware_interface/EffortJointInterface</hardwareInterface>
       </joint>
       <actuator name="${prefix}joint_4">
@@ -225,5 +284,5 @@
       <type>transmission_interface/SimpleTransmission</type>
       <joint name="${prefix}joint_5">
-        <hardwareInterface>hardware_interface/PositionJointInterface</hardwareInterface>
+        <hardwareInterface>hardware_interface/EffortJointInterface</hardwareInterface>
       </joint>
       <actuator name="${prefix}joint_5">
@@ -234,7 +293,16 @@
       <type>transmission_interface/SimpleTransmission</type>
       <joint name="${prefix}joint_6">
-        <hardwareInterface>hardware_interface/PositionJointInterface</hardwareInterface>
+        <hardwareInterface>hardware_interface/EffortJointInterface</hardwareInterface>
       </joint>
       <actuator name="${prefix}joint_6">
+        <mechanicalReduction>1</mechanicalReduction>
+      </actuator>
+    </transmission>
+		<transmission name="${prefix}end_joint_trans">
+      <type>transmission_interface/SimpleTransmission</type>
+      <joint name="${prefix}end_joint">
+        <hardwareInterface>hardware_interface/EffortJointInterface</hardwareInterface>
+      </joint>
+      <actuator name="${prefix}end_joint">
         <mechanicalReduction>1</mechanicalReduction>
       </actuator>
